Commit message: Put Fanuc in pick and place example

File: tesseract_ros/tesseract_examples/tesseract_ros_examples/urdf/environment.xacro (robot description, xacro)
@@ -1,4 +1,4 @@
 <?xml version="1.0" ?>
-<robot name="environment" xmlns:xacro="http://www.ros.org/wiki/xacro">
+<robot name="environment" xmlns:xacro="http://wiki.ros.org/xacro">
 <xacro:macro name="workcell" params="parent_link *location">
   <material name="light_gray">

File: tesseract_ros/tesseract_examples/tesseract_ros_examples/urdf/pick_and_place_plan.xacro (robot description, xacro)
@@ -1,4 +1,4 @@
 <?xml version="1.0" ?>
-<robot name="robot" xmlns:xacro="http://www.ros.org/wiki/xacro">
+<robot name="pm" xmlns:xacro="http://wiki.ros.org/xacro">
     <!-- Create links -->
     <link name="world"/>
@@ -7,9 +7,9 @@
     <xacro:include filename="$(find tesseract_ros_examples)/urdf/iiwa7/materials.xacro" />
     <!--Import the lbr iiwa macro -->
-    <xacro:include filename="$(find tesseract_ros_examples)/urdf/iiwa7/iiwa7.xacro"/>
+    <!-- <xacro:include filename="$(find tesseract_ros_examples)/urdf/pm.xacro"/> -->
+    <xacro:include filename="$(find pm_description)/urdf/m20ib25c_macro.xacro"/>
     <!-- Include robot -->
-    <xacro:iiwa7 hardware_interface="PositionJointInterface" robot_name="iiwa" parent="base_link">
-        <origin xyz="0.0 0 0.0" rpy="0 0 0"/>
-    </xacro:iiwa7>
+    <!-- <xacro:pm prefix="arm_"/> -->
+    <xacro:fanuc_m20ib25c prefix="arm_"/>
     <!-- Include workcell (creates joint from world to workcell_base)-->
     <xacro:include filename="$(find tesseract_ros_examples)/urdf/environment.xacro"/>
@@ -26,3 +26,8 @@
       <origin xyz="0 -0.0381 0.00953" rpy="0 0 1.5708"/>
     </joint>
+    <joint name="base_link_robot" type="fixed">
+        <parent link="base_link"/>
+        <child link="arm_base_link"/>
+        <origin xyz="0.0 0.0 0.0" rpy="0 0 0"/>
+    </joint>
 </robot>

Commit message: Basic trajectory generation for fanuc

File: tesseract_ros/tesseract_examples/tesseract_ros_examples/urdf/environment.xacro (robot description, xacro)
@@ -9,45 +9,15 @@
   </material>
   <link name="workcell_base">
-    <visual>
+    <visual name="workcell_table">
       <geometry>
-        <mesh filename="package://tesseract_ros_examples/meshes/pick_and_place/workcell.STL"/>
+        <box size="1.0 2.0 0.77153"/>
       </geometry>
-      <material name="light_gray"/>
+      <origin xyz="0.0 0.3 -0.385765"/>
     </visual>
     <collision name="workcell_table">
       <geometry>
-        <box size="0.8 1.25 0.77153"/>
+        <box size="1.0 2.0 0.77153"/>
       </geometry>
       <origin xyz="0.0 0.3 -0.385765"/>
-    </collision>
-    <collision name="workcell_columnSW">
-      <geometry>
-        <box size="0.1 0.1 1.25"/>
-      </geometry>
-      <origin xyz="-.3302 -.2794 0.6"/>
-    </collision>
-    <collision name="workcell_columnsSE">
-      <geometry>
-        <box size="0.1 0.1 1.25"/>
-      </geometry>
-      <origin xyz=".3302 -.2794 0.6"/>
-    </collision>
-    <collision name="workcell_columnNW">
-      <geometry>
-        <box size="0.1 0.1 1.25"/>
-      </geometry>
-      <origin xyz="-.3302 0.8382 0.6"/>colors
-    </collision>
-    <collision name="workcell_columnNE">
-      <geometry>
-        <box size="0.1 0.1 1.25"/>
-      </geometry>
-      <origin xyz=".3302 0.8382 0.6"/>
-    </collision>
-    <collision name="workcell_top">
-      <geometry>
-        <box size="0.95 1.4 0.2"/>
-      </geometry>
-      <origin xyz="0.0 0.3 1.2"/>
     </collision>
   </link>
@@ -61,15 +31,45 @@
 <xacro:macro name="cabinet" params="id parent_link *location">
   <link name="cabinet_${id}">
-<collision name="cabinet_${id}_back">
-  <geometry>
-    <box size="0.5969 0.0254 0.762"/>
-  </geometry>
-  <origin xyz=".2985 -.0127 -0.381"/>
-</collision>
+    <visual name="cabinet_${id}_sideL">
+      <geometry>
+        <box size="0.0254 0.3048 0.762"/>
+      </geometry>
+      <origin xyz=".0127 0.5524 -0.381"/>
+    </visual>
+    <visual name="cabinet_${id}_sideR">
+      <geometry>
+        <box size="0.0254 0.3048 0.762"/>
+      </geometry>
+      <origin xyz=".5969 0.5524 -0.381"/>
+    </visual>
+    <visual name="cabinet_${id}_cabinet1">
+      <geometry>
+        <box size="0.5969 0.3048 0.0254"/>
+      </geometry>
+      <origin xyz=".2985 0.5524  -0.7493"/>
+    </visual>
+    <visual name="cabinet_${id}_cabinet2">
+      <geometry>
+        <box size="0.5969 0.3048 0.0254"/>
+      </geometry>
+      <origin xyz=".2985 0.5524  -0.508"/>
+    </visual>
+    <visual name="cabinet_${id}_cabinet3">
+      <geometry>
+        <box size="0.5969 0.3048 0.0254"/>
+      </geometry>
+      <origin xyz=".2985 0.5524  -0.254"/>
+    </visual>
+    <visual name="cabinet_${id}_cabinet4">
+      <geometry>
+        <box size="0.5969 0.3048 0.0254"/>
+      </geometry>
+      <origin xyz=".2985 0.5524  -0.0127"/>
+    </visual>
 <collision name="cabinet_${id}_sideL">
   <geometry>
     <box size="0.0254 0.3048 0.762"/>
   </geometry>
-  <origin xyz="0.0127 -0.1524 -0.381"/>
+  <origin xyz=".0127 0.5524 -0.381"/>
 </collision>
 <collision name="cabinet_${id}_sideR">
@@ -77,5 +77,5 @@
   <box size="0.0254 0.3048 0.762"/>
 </geometry>
-<origin xyz="0.5969 -0.1524 -0.381"/>
+<origin xyz=".5969 0.5524 -0.381"/>
 </collision>
 <collision name="cabinet_${id}_cabinet1">
@@ -83,5 +83,5 @@
           <box size="0.5969 0.3048 0.0254"/>
     </geometry>
-    <origin xyz=".2985 -0.1524  -0.7493"/>
+    <origin xyz=".2985 0.5524  -0.7493"/>
 </collision>
 <collision name="cabinet_${id}_cabinet2">
@@ -89,5 +89,5 @@
         <box size="0.5969 0.3048 0.0254"/>
     </geometry>
-    <origin xyz=".2985 -0.1524  -0.508"/>
+    <origin xyz=".2985 0.5524  -0.508"/>
 </collision>
 <collision name="cabinet_${id}_cabinet3">
@@ -95,5 +95,5 @@
         <box size="0.5969 0.3048 0.0254"/>
     </geometry>
-    <origin xyz=".2985 -0.1524  -0.254"/>
+    <origin xyz=".2985 0.5524  -0.254"/>
 </collision>
 <collision name="cabinet_${id}_cabinet4">
@@ -101,5 +101,5 @@
         <box size="0.5969 0.3048 0.0254"/>
     </geometry>
-    <origin xyz=".2985 -0.1524  -0.0127"/>
+    <origin xyz=".2985 0.5524  -0.0127"/>
 </collision>
   </link>
